File: pcb/CMD.kicad_sch (KiCad schematic)
At the start: 87 parts, among them J1 Conn_01x06_Pin, J2 Conn_01x06_Socket

Commit message: Adapt vendor(id)
Parts:
- J1: Vendor DigiKey -> HTL; VendorId 952-3235-ND -> 103666
- J2: Vendor DigiKey -> HTL; VendorId 952-3199-1-ND -> 103667
Changed lines of the file:
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@@
       (effects (font (size 1.27 1.27)) hide)
     )
-    (property "Vendor" "DigiKey" (at 21.59 33.02 0)
-      (effects (font (size 1.27 1.27)) hide)
-    )
-    (property "VendorId" "952-3235-ND" (at 21.59 33.02 0)
+    (property "Vendor" "HTL" (at 21.59 33.02 0)
+      (effects (font (size 1.27 1.27)) hide)
+    )
+    (property "VendorId" "103666" (at 21.59 33.02 0)
       (effects (font (size 1.27 1.27)) hide)
     )
@@
       (effects (font (size 1.27 1.27)) hide)
     )
-    (property "Vendor" "DigiKey" (at 69.85 33.02 0)
-      (effects (font (size 1.27 1.27)) hide)
-    )
-    (property "VendorId" "952-3199-1-ND" (at 69.85 33.02 0)
-      (effects (font (size 1.27 1.27)) hide)
-    )
+    (property "Vendor" "HTL" (at 69.85 33.02 0)
+      (effects (font (size 1.27 1.27)) hide)
+    )
+    (property "VendorId" "103667" (at 69.85 33.02 0)
+      (effects (font (size 1.27 1.27)) hide)
+    )
